Commit message: switch to xarm gripper from DH_AG95 gripper

File: scout_xarm_grip_moveit_config/config/scout_xarm_gripper.xacro (robot description, xacro)
@@ -34,5 +34,4 @@
         link="base_link" />
     </joint>
-    <!-- Load xarm gripper attached to link_eef -->
     <xacro:load_gripper attach_to="link_eef" effort_control="$(arg effort_control)" velocity_control="$(arg velocity_control)"/>
     <joint
@@ -58,10 +57,3 @@
         link="box_link" />
     </joint>
-    <!-- Create a new end effector link for MoveIt interactive marker -->
-    <link name="moveit_eef"/>
-    <joint name="moveit_eef_joint" type="fixed">
-      <origin rpy="0 0 0" xyz="0.0 0.0 0.2"/>
-      <parent link="link_eef"/>
-      <child link="moveit_eef"/>
-    </joint>
     </robot>
