Commit message: add link to correct the plan target

File: src/scout_xarm_gripper.xacro (robot description, xacro)
@@ -68,3 +68,10 @@
         link="box_link" />
     </joint>
+    <!-- Create a new end effector link for MoveIt interactive marker -->
+    <link name="moveit_eef"/>
+    <joint name="moveit_eef_joint" type="fixed">
+      <origin rpy="0 0 0" xyz="0.0 0.0 0.2"/>
+      <parent link="link_eef"/>
+      <child link="moveit_eef"/>
+    </joint>
     </robot>

Commit message: update move_node with approach vector, copy moveit config pkg, update xacro

File: src/scout_xarm_gripper.xacro (robot description, xacro)
@@ -71,5 +71,5 @@
     <link name="moveit_eef"/>
     <joint name="moveit_eef_joint" type="fixed">
-      <origin rpy="0 0 0" xyz="0.0 0.0 0.2"/>
+      <origin rpy="3.14 -1.57 0" xyz="0.0 0.0 0.17"/>
       <parent link="link_eef"/>
       <child link="moveit_eef"/>
